File: _autosave-nes_power_video.kicad_pcb (KiCad board)
At the start: 2 copper layers, 59.9 x 59.7 mm, 13 parts, among them J2 Audio, J3 Video, J4 Conn_01x05, Q1 2SA1015

Commit message: Changing to proper RCA jacks. Also getting ready for V2.
Parts:
- moved J3 0.20 mm to (69.0, 68.8)
Routing:
- net /5V: track 186.6 -> 238.6 mm
- net Net-(J2-TIP): track 14.5 -> 48.5 mm
- net Net-(USB-C1-CC2): track 0.00 -> 31.1 mm
- net Net-(C2-Pad2): track 0.00 -> 24.8 mm
- net /raw_5v: track 4.22 -> 12.9 mm
- net GND: track 13.3 -> 11.6 mm, vias 5 -> 4
- net unconnected-(J3-SHUNT-Pad3): vias 1 -> 0
